File: Tests/7730TestPlatform/7730TestPlatform.kicad_sch (KiCad schematic)
At the start: 66 parts, among them J1 Conn_01x06_Male, J2 AudioJack4, J3 Conn_01x12_Male, J4 Conn_01x04_Male, J5 Conn_Coaxial, J6 Conn_01x02_Male, J7 Conn_01x19_Female, U1 SAF7730HV/336, Y1 41.6M

Commit message: Finish Test Platform
Parts:
- removed C12, C13, C16: 3.3n NPO, Capacitor_SMD:C_0603_1608Metric_Pad1.08x0.95mm_HandSolder, symbol Device:C
- removed FB1: BLM41PG102SN1, Inductor_SMD:L_1806_4516Metric_Pad1.45x1.90mm_HandSolder, symbol Device:FerriteBead
- added BT1: 3.7V LiPo, Connector_Molex:Molex_KK-254_AE-6410-02A_1x02_P2.54mm_Vertical, symbol Device:Battery_Cell
- added C36: 10uF, Capacitor_SMD:CP_Elec_4x5.4, symbol Device:C_Polarized
- added C37: 10n, Capacitor_SMD:C_0603_1608Metric_Pad1.08x0.95mm_HandSolder, symbol Device:C_Small
- added C38: 27n, Capacitor_SMD:C_0603_1608Metric_Pad1.08x0.95mm_HandSolder, symbol Device:C
- added C39: 150p, Capacitor_SMD:C_0603_1608Metric_Pad1.08x0.95mm_HandSolder, symbol Device:C
- added C40: 81p, Capacitor_SMD:C_0603_1608Metric_Pad1.08x0.95mm_HandSolder, symbol Device:C
- added C41: 20u, Capacitor_SMD:CP_Elec_4x5.4, symbol Device:C_Polarized
- added C42, C45: 10u, Capacitor_SMD:CP_Elec_4x5.4, symbol Device:C_Polarized
- added C43: 100n, Capacitor_SMD:C_0603_1608Metric_Pad1.08x0.95mm_HandSolder, symbol Device:C
- added C44: 33u Tantalum, Capacitor_Tantalum_SMD:CP_EIA-3528-21_Kemet-B_Pad1.50x2.35mm_HandSolder, symbol Device:C_Polarized
- added D1: MBRS130LT(MA728), Diode_SMD:D_SOD-323_HandSoldering, symbol Device:D_Schottky
- added L2: 8.1uH, Inductor_SMD:L_Taiyo-Yuden_MD-4040, symbol Device:L
- added R13: 6k, Resistor_SMD:R_0603_1608Metric_Pad0.98x0.95mm_HandSolder, symbol Device:R
- added R14: 68k, Resistor_SMD:R_0603_1608Metric_Pad0.98x0.95mm_HandSolder, symbol Device:R
- added R15: 400k, Resistor_SMD:R_0603_1608Metric_Pad0.98x0.95mm_HandSolder, symbol Device:R
- added U2: LT1763-1.8, Package_SO:SO-8_3.9x4.9mm_P1.27mm, symbol Regulator_Linear:LT1763-1.8
- added U3: MAX1790, max1790:max1790eua, symbol Converter_DCDC:MAX1790
- added U4: LT1764-3.3, Package_TO_SOT_SMD:TO-263-5_TabPin3, symbol Regulator_Linear:LT1764-3.3
- C17: footprint (none) -> Capacitor_SMD:CP_Elec_6.3x5.4_Nichicon
- C18: footprint (none) -> Capacitor_SMD:CP_Elec_10x10
- C2, C20, C30, C32, C35, C6: footprint (none) -> Capacitor_SMD:CP_Elec_4x5.4
- J1: footprint (none) -> Connector_PinHeader_2.54mm:PinHeader_1x06_P2.54mm_Vertical
- J2: footprint (none) -> Connector_Audio:Jack_3.5mm_PJ320D_Horizontal
- J3: footprint (none) -> Connector_PinHeader_2.54mm:PinHeader_1x12_P2.54mm_Vertical
- J4: footprint (none) -> Connector_PinHeader_2.54mm:PinHeader_1x04_P2.54mm_Vertical
- J5: footprint (none) -> Connector_Coaxial:SMA_Amphenol_901-143_Horizontal
- J6: footprint (none) -> Connector_PinHeader_2.54mm:PinHeader_1x02_P2.54mm_Vertical
- J7: footprint (none) -> Connector_PinSocket_2.54mm:PinSocket_1x19_P2.54mm_Vertical
- J8: renamed from J?; footprint (none) -> Connector_Audio:Jack_3.5mm_CUI_SJ1-3533NG_Horizontal
- Y1: footprint (none) -> Crystal:Crystal_SMD_5032-2Pin_5.0x3.2mm_HandSoldering
Connections:
- net +1V8: now also C36.1, C37.1, U2.1 (OUT), U2.2 (SENSE)
- net +3V3: now also C45.1, U4.4 (OUT), U4.5 (SENSE)
- net +8V5: now also C43.1, C44.1, D1.1 (K), R15.1
- net GND: now also BT1.2 (-), C36.2, C38.1, C39.2, C40.2, C41.2, C42.2, C43.2, C44.2, C45.2, R14.2, U2.3 (GND), U2.6 (GND), U2.7 (GND), U3.4 (GND), U4.3 (GND); no longer C11.2, J2.R1, U1.38 (DACRR), U1.43 (DAC_FR)
- net VDDD: now also U1.94 (VDDD3); no longer U1.g4 (VDDD3)
- net at J1.3 (Pin_3), R7.2, U1.28 (SCL): no longer J1.4 (Pin_4), R8.2, U1.29 (SDA)
- net at C6.2, C7.1: now also R5.2, U1.11 (VREFAD), U1.12 (CD_R), U1.13 (CD_R_GND), U1.14 (CD_L_GND), U1.15 (CD_L), U1.16 (PHONE_IN), U1.17 (PHONEGND), U1.18 (NAV), U1.19 (NAV_GND)
- net at C5.2, R4.2, U1.5 (AUX_L): now also R1.2
- net at J3.4 (Pin_4): now also U1.99 (TDsP_IOF4); no longer U1.g9 (TDsP_IOF4)
- net at C3.2: now also R1.1
- net IFP: now reaches J7.15 (Pin_15), U1.143 (IFADP2)
- net IFN: now reaches J7.16 (Pin_16), U1.144 (IFADN2)
- new net: R14.1, R15.2, U3.2 (FB)
- new net: D1.2 (A), L2.2, U3.5 (LX)
- new net: J1.4 (Pin_4), R8.2, U1.29 (SDA)
- new net: C40.1, R13.2
- new net: C39.1, R13.1, U3.1 (COMP)
- new net: C37.2, U2.4 (BYP)
- new net: C11.2, J2.R1, U1.38 (DACRR), U1.43 (DAC_FR)
- new net: C38.2, U3.8 (SS)
- new net Bat: BT1.1 (+), C41.1, C42.1, L2.1, U2.5 (~{SHDN}), U2.8 (IN), U3.3 (~{SHDN), U3.6 (IN), U4.1 (~{SHDN}), U4.2 (IN)
- no-connect marks 3 -> 4
Other:
- moved on the sheet: C6, C7
